File: KiCad_Project/2022/Projects/ADNS-9800/ADNS-9800.kicad_sch (KiCad schematic)
At the start: 15 parts

Commit message: 徹夜の進捗、朝マック食べに行きます
Parts:
- removed R1, R2: (no value), symbol Device:R
- C1, C5, C7: value (none) -> 100nF (0.1uF); footprint (none) -> Capacitor_SMD:C_0603_1608Metric_Pad1.08x0.95mm_HandSolder
- C2: value (none) -> 1uF; footprint (none) -> Capacitor_SMD:C_0603_1608Metric_Pad1.08x0.95mm_HandSolder
- C3: value (none) -> 470pF; footprint (none) -> Capacitor_SMD:C_0603_1608Metric_Pad1.08x0.95mm_HandSolder
- C4, C9: value (none) -> 10uF; footprint (none) -> Capacitor_SMD:C_0603_1608Metric_Pad1.08x0.95mm_HandSolder
- C6: value (none) -> 100nF; footprint (none) -> Capacitor_SMD:C_0603_1608Metric_Pad1.08x0.95mm_HandSolder
- C8: value (none) -> 3.3uF; footprint (none) -> Capacitor_SMD:C_0603_1608Metric_Pad1.08x0.95mm_HandSolder
- J1: value (none) -> Conn_01x04; footprint (none) -> Connector_JST:JST_XH_S4B-XH-A_1x04_P2.50mm_Horizontal
- Q1: value (none) -> IRLML6402; footprint (none) -> Package_TO_SOT_SMD:SOT-23
- U$1: value (none) -> AVAGO_ADNS-9500; footprint (none) -> ADNS-9800:AVAGO_ADNS-9500
- U1: value (none) -> SeeeduinoXIAO; footprint (none) -> Library:Seeeduino XIAO-MOUDLE14P-2.54-21X17.8MM
