File: KiCad_Project/2022/Projects/Main_Board/Main_Board.kicad_pcb (KiCad board)
At the start: 2 copper layers, 120 x 113 mm, 58 parts, among them J1 Conn_01x02, J10 Conn_01x04, J11 Conn_01x06, J12 Conn_01x02, J13 Conn_01x04, J14 Conn_01x02, J15 Conn_01x03, J16 Conn_01x07, J2 Conn_01x03, J3 Conn_01x08, J4 Conn_01x03, J5 USB_B_Micro, J6 Conn_01x04, J7 Conn_01x04, J8 Conn_01x04, J9 Conn_01x04, SW1 SW_Push, SW11 SW_SPST, SW2 SW_SPST, SW5 SW_SPST, SW6 SW_DIP_x01, SW7 SW_Push, SW8 SW_Push, SW9 SW_Push, U1 Stamp_Pico, U2 SeeeduinoXIAO, U3 Teensy4.0, U4 SeeeduinoXIAO, U5 OpenMV, U6 LF33_TO252, U7 module_mpu6050, U8 Akizuki_Logiv_Level_converter

Commit message: レジストを抜いて文字とURLを記入
Other:
- board text added: "MUNAKO_Hercules"
- board text added: "Main_Board Ver.2022 Designed by Kiyo"
- board text added: "https://github.com/MUNAKATA-EPC"
Changed lines of the file:
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@@
     )
     (pad_to_mask_clearance 0)
-    (grid_origin 250.782005 68.984651)
+    (grid_origin 190.782005 149.24201)
     (pcbplotparams
       (layerselection 0x00010fc_ffffffff)
@@
   (gr_circle (center 190.782 95.596011) (end 220.782 95.596011) (layer "User.1") (width 0.1) (fill none))
   (gr_rect (start 130.782005 68.984651) (end 144.782005 113.984651) (layer "User.1") (width 0.1) (fill none))
+  (gr_text "Main_Board\nVer.2022\nDesigned by Kiyo" (at 142.522005 80.66201 270) (layer "F.Mask")
+    (effects (font (size 1.5 1.5) (thickness 0.3)))
+  )
+  (gr_text "MUNAKO_Hercules" (at 190.782005 152.499851) (layer "F.Mask")
+    (effects (font (size 2 2) (thickness 0.3)))
+  )
+  (gr_text "https://github.com/MUNAKATA-EPC" (at 241.582005 93.36201 90) (layer "F.Mask")
+    (effects (font (size 1.5 1.5) (thickness 0.3)))
+  )
   (segment (start 173.9347 114.7261) (end 190.317 114.7261) (width 0.25) (layer "F.Cu") (net 1))
   (segment (start 217.1343 126.2131) (end 220.656 126.2131) (width 0.25) (layer "F.Cu") (net 1))
